Commit message: Fix robot arm description

File: robot_description/urdf/mecharm_270_pi_adaptive_gripper.urdf (robot description, URDF)
Before this commit: robot firefighter, 14 links, 13 joints
Joints:
- removed joint gripper_controller
- added joint zgripper_joint: type revolute, parent gripper_base, child gripper_left3, origin xyz=-0.012 0.005 0 rpy=0 0 0, axis 0 0 1, limit lower=-0.74 upper=0.15 effort=1000.0 velocity=20
- joint gripper_base_to_gripper_left2: limit lower=-0.8 upper=0.5 effort=1000.0 velocity=0 -> lower=-0.8 upper=0.5 effort=1000.0 velocity=20; mimic joint=gripper_controller multiplier=1.0 offset=0 -> joint=zgripper_joint multiplier=1.0 offset=0
- joint gripper_base_to_gripper_right2: limit lower=-0.5 upper=0.8 effort=1000.0 velocity=0 -> lower=-0.5 upper=0.8 effort=1000.0 velocity=20; mimic joint=gripper_controller multiplier=-1.0 offset=0 -> joint=zgripper_joint multiplier=-1.0 offset=0
- joint gripper_base_to_gripper_right3: limit lower=-0.15 upper=0.7 effort=1000.0 velocity=0 -> lower=-0.15 upper=0.7 effort=1000.0 velocity=20; mimic joint=gripper_controller multiplier=-1.0 offset=0 -> joint=zgripper_joint multiplier=-1.0 offset=0
- joint gripper_left3_to_gripper_left1: limit lower=-0.5 upper=0.5 effort=1000.0 velocity=0 -> lower=-0.5 upper=0.5 effort=1000.0 velocity=20; mimic joint=gripper_controller multiplier=-1.0 offset=0 -> joint=zgripper_joint multiplier=-1.0 offset=0
- joint gripper_right3_to_gripper_right1: limit lower=-0.5 upper=0.5 effort=1000.0 velocity=0 -> lower=-0.5 upper=0.5 effort=1000.0 velocity=20; mimic joint=gripper_controller multiplier=1.0 offset=0 -> joint=zgripper_joint multiplier=1.0 offset=0
- joint joint1_to_base: limit lower=-2.792527 upper=2.792527 effort=1000.0 velocity=0 -> lower=-2.792527 upper=2.792527 effort=1000.0 velocity=20
- joint joint2_to_joint1: limit lower=-1.3089 upper=2.0943 effort=1000.0 velocity=0 -> lower=-1.3089 upper=2.0943 effort=1000.0 velocity=20
- joint joint3_to_joint2: limit lower=-3.0543 upper=1.1344 effort=1000.0 velocity=0 -> lower=-3.0543 upper=1.1344 effort=1000.0 velocity=20
- joint joint4_to_joint3: limit lower=-2.7052 upper=2.7052 effort=1000.0 velocity=0 -> lower=-2.7052 upper=2.7052 effort=1000.0 velocity=20
- joint joint5_to_joint4: limit lower=-2.0071 upper=2.0071 effort=1000.0 velocity=0 -> lower=-2.0071 upper=2.0071 effort=1000.0 velocity=20
- joint joint6_to_joint5: limit lower=-3.14 upper=3.14 effort=1000.0 velocity=0 -> lower=-3.14 upper=3.14 effort=1000.0 velocity=20
